File: PCBs/input-selector/input-selector.sch (KiCad schematic (older format))
At the start: 46 parts, among them J1 Conn_01x06_Male, K1 IM40, K2 IM40, K3 IM40, K4 IM40, K5 IM40, K6 IM40, U1 ULN2003, U2 MCP23S17_SO, U3 ULN2003

Commit message: Fixing input selector panasonic relay footprint
Parts:
- K1, K2, K3, K4, K5, K6, MUTE1: footprint w_relay:relay_gq-pth -> panasonic-relay:gq-th
Changed lines of the file:
@@
 F 0 "MUTE1" H 11730 8096 50  0000 L CNN
 F 1 "IM01" H 11730 8005 50  0000 L CNN
-F 2 "w_relay:relay_gq-pth" H 10900 8050 50  0001 C CNN
+F 2 "panasonic-relay:gq-th" H 10900 8050 50  0001 C CNN
 F 3 "http://www.te.com/commerce/DocumentDelivery/DDEController?Action=srchrtrv&DocNm=108-98001&DocType=SS&DocLang=EN" H 10900 8050 50  0001 C CNN
 	1    11100 8050
@@
 F 0 "K2" H 11730 2946 50  0000 L CNN
 F 1 "IM40" H 11730 2855 50  0000 L CNN
-F 2 "w_relay:relay_gq-pth" H 10900 2900 50  0001 C CNN
+F 2 "panasonic-relay:gq-th" H 10900 2900 50  0001 C CNN
 F 3 "http://www.te.com/commerce/DocumentDelivery/DDEController?Action=srchrtrv&DocNm=108-98001&DocType=SS&DocLang=EN" H 10900 2900 50  0001 C CNN
 	1    11100 2900
@@
 F 0 "K1" H 11730 1946 50  0000 L CNN
 F 1 "IM40" H 11730 1855 50  0000 L CNN
-F 2 "w_relay:relay_gq-pth" H 10900 1900 50  0001 C CNN
+F 2 "panasonic-relay:gq-th" H 10900 1900 50  0001 C CNN
 F 3 "http://www.te.com/commerce/DocumentDelivery/DDEController?Action=srchrtrv&DocNm=108-98001&DocType=SS&DocLang=EN" H 10900 1900 50  0001 C CNN
 	1    11100 1900
@@
 F 0 "K3" H 11730 3946 50  0000 L CNN
 F 1 "IM40" H 11730 3855 50  0000 L CNN
-F 2 "w_relay:relay_gq-pth" H 10900 3900 50  0001 C CNN
+F 2 "panasonic-relay:gq-th" H 10900 3900 50  0001 C CNN
 F 3 "http://www.te.com/commerce/DocumentDelivery/DDEController?Action=srchrtrv&DocNm=108-98001&DocType=SS&DocLang=EN" H 10900 3900 50  0001 C CNN
 	1    11100 3900
@@
 F 0 "K4" H 11730 4946 50  0000 L CNN
 F 1 "IM40" H 11730 4855 50  0000 L CNN
-F 2 "w_relay:relay_gq-pth" H 10900 4900 50  0001 C CNN
+F 2 "panasonic-relay:gq-th" H 10900 4900 50  0001 C CNN
 F 3 "http://www.te.com/commerce/DocumentDelivery/DDEController?Action=srchrtrv&DocNm=108-98001&DocType=SS&DocLang=EN" H 10900 4900 50  0001 C CNN
 	1    11100 4900
@@
 F 0 "K5" H 11730 5946 50  0000 L CNN
 F 1 "IM40" H 11730 5855 50  0000 L CNN
-F 2 "w_relay:relay_gq-pth" H 10900 5900 50  0001 C CNN
+F 2 "panasonic-relay:gq-th" H 10900 5900 50  0001 C CNN
 F 3 "http://www.te.com/commerce/DocumentDelivery/DDEController?Action=srchrtrv&DocNm=108-98001&DocType=SS&DocLang=EN" H 10900 5900 50  0001 C CNN
 	1    11100 5900
@@
 F 0 "K6" H 11730 6946 50  0000 L CNN
 F 1 "IM40" H 11730 6855 50  0000 L CNN
-F 2 "w_relay:relay_gq-pth" H 10900 6900 50  0001 C CNN
+F 2 "panasonic-relay:gq-th" H 10900 6900 50  0001 C CNN
 F 3 "http://www.te.com/commerce/DocumentDelivery/DDEController?Action=srchrtrv&DocNm=108-98001&DocType=SS&DocLang=EN" H 10900 6900 50  0001 C CNN
 	1    11100 6900

Commit message: Switching relay type to Omron G6J relays
Since I can't find a source for the others
Parts:
- K1, K2, K3, K4, K5, K6, MUTE1: footprint panasonic-relay:gq-th -> omron-relay:g6j-2p-y
Changed lines of the file:
@@
 F 0 "MUTE1" H 11730 8096 50  0000 L CNN
 F 1 "IM01" H 11730 8005 50  0000 L CNN
-F 2 "panasonic-relay:gq-th" H 10900 8050 50  0001 C CNN
+F 2 "omron-relay:g6j-2p-y" H 10900 8050 50  0001 C CNN
 F 3 "http://www.te.com/commerce/DocumentDelivery/DDEController?Action=srchrtrv&DocNm=108-98001&DocType=SS&DocLang=EN" H 10900 8050 50  0001 C CNN
 	1    11100 8050
@@
 F 0 "K2" H 11730 2946 50  0000 L CNN
 F 1 "IM40" H 11730 2855 50  0000 L CNN
-F 2 "panasonic-relay:gq-th" H 10900 2900 50  0001 C CNN
+F 2 "omron-relay:g6j-2p-y" H 10900 2900 50  0001 C CNN
 F 3 "http://www.te.com/commerce/DocumentDelivery/DDEController?Action=srchrtrv&DocNm=108-98001&DocType=SS&DocLang=EN" H 10900 2900 50  0001 C CNN
 	1    11100 2900
@@
 F 0 "K1" H 11730 1946 50  0000 L CNN
 F 1 "IM40" H 11730 1855 50  0000 L CNN
-F 2 "panasonic-relay:gq-th" H 10900 1900 50  0001 C CNN
+F 2 "omron-relay:g6j-2p-y" H 10900 1900 50  0001 C CNN
 F 3 "http://www.te.com/commerce/DocumentDelivery/DDEController?Action=srchrtrv&DocNm=108-98001&DocType=SS&DocLang=EN" H 10900 1900 50  0001 C CNN
 	1    11100 1900
@@
 F 0 "K3" H 11730 3946 50  0000 L CNN
 F 1 "IM40" H 11730 3855 50  0000 L CNN
-F 2 "panasonic-relay:gq-th" H 10900 3900 50  0001 C CNN
+F 2 "omron-relay:g6j-2p-y" H 10900 3900 50  0001 C CNN
 F 3 "http://www.te.com/commerce/DocumentDelivery/DDEController?Action=srchrtrv&DocNm=108-98001&DocType=SS&DocLang=EN" H 10900 3900 50  0001 C CNN
 	1    11100 3900
@@
 F 0 "K4" H 11730 4946 50  0000 L CNN
 F 1 "IM40" H 11730 4855 50  0000 L CNN
-F 2 "panasonic-relay:gq-th" H 10900 4900 50  0001 C CNN
+F 2 "omron-relay:g6j-2p-y" H 10900 4900 50  0001 C CNN
 F 3 "http://www.te.com/commerce/DocumentDelivery/DDEController?Action=srchrtrv&DocNm=108-98001&DocType=SS&DocLang=EN" H 10900 4900 50  0001 C CNN
 	1    11100 4900
@@
 F 0 "K5" H 11730 5946 50  0000 L CNN
 F 1 "IM40" H 11730 5855 50  0000 L CNN
-F 2 "panasonic-relay:gq-th" H 10900 5900 50  0001 C CNN
+F 2 "omron-relay:g6j-2p-y" H 10900 5900 50  0001 C CNN
 F 3 "http://www.te.com/commerce/DocumentDelivery/DDEController?Action=srchrtrv&DocNm=108-98001&DocType=SS&DocLang=EN" H 10900 5900 50  0001 C CNN
 	1    11100 5900
@@
 F 0 "K6" H 11730 6946 50  0000 L CNN
 F 1 "IM40" H 11730 6855 50  0000 L CNN
-F 2 "panasonic-relay:gq-th" H 10900 6900 50  0001 C CNN
+F 2 "omron-relay:g6j-2p-y" H 10900 6900 50  0001 C CNN
 F 3 "http://www.te.com/commerce/DocumentDelivery/DDEController?Action=srchrtrv&DocNm=108-98001&DocType=SS&DocLang=EN" H 10900 6900 50  0001 C CNN
 	1    11100 6900

Commit message: adding BoMs, images and small design updates
Parts:
- renumbered C1 to C4
Changed lines of the file:
@@
 $EndComp
 $Comp
-L Device:C C1
+L Device:C C4
 U 1 1 5C3FB3EC
 P 3750 2400
-F 0 "C1" H 3865 2446 50  0000 L CNN
+F 0 "C4" H 3865 2446 50  0000 L CNN
 F 1 "C" H 3865 2355 50  0000 L CNN
 F 2 "Capacitor_SMD:C_1206_3216Metric_Pad1.42x1.75mm_HandSolder" H 3788 2250 50  0001 C CNN
