File: PCBs/input-selector/input-selector.kicad_pcb (KiCad board)
At the start: 2 copper layers, 90.2 x 52.1 mm, 46 parts, among them J1 Conn_01x06_Male, K1 IM40, K2 IM40, K3 IM40, K4 IM40, K5 IM40, K6 IM40, U1 ULN2003, U2 MCP23S17_SO, U3 ULN2003

Commit message: adding BoMs, images and small design updates (#4)
Parts:
- removed C1: C, Capacitor_SMD:C_1206_3216Metric_Pad1.42x1.75mm_HandSolder
- added C4: C, Capacitor_SMD:C_1206_3216Metric_Pad1.42x1.75mm_HandSolder, B.Cu at (125.2, 106.7)
Other:
- board text added: "Input Selector v3.0"
- board text added: "v3.0"
Changed lines of the file:
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@@
   (general
     (thickness 1.6)
-    (drawings 25)
+    (drawings 29)
     (tracks 343)
     (zones 0)
@@
   (page A4)
   (layers
-    (0 F.Cu signal)
+    (0 F.Cu signal hide)
     (31 B.Cu signal)
-    (32 B.Adhes user)
-    (33 F.Adhes user)
+    (32 B.Adhes user hide)
+    (33 F.Adhes user hide)
     (34 B.Paste user)
-    (35 F.Paste user)
+    (35 F.Paste user hide)
     (36 B.SilkS user)
-    (37 F.SilkS user)
+    (37 F.SilkS user hide)
     (38 B.Mask user)
-    (39 F.Mask user)
-    (40 Dwgs.User user)
-    (41 Cmts.User user)
-    (42 Eco1.User user)
-    (43 Eco2.User user)
+    (39 F.Mask user hide)
+    (40 Dwgs.User user hide)
+    (41 Cmts.User user hide)
+    (42 Eco1.User user hide)
+    (43 Eco2.User user hide)
     (44 Edge.Cuts user)
-    (45 Margin user)
+    (45 Margin user hide)
     (46 B.CrtYd user)
-    (47 F.CrtYd user)
+    (47 F.CrtYd user hide)
     (48 B.Fab user)
-    (49 F.Fab user)
+    (49 F.Fab user hide)
   )
   (setup
@@
     (add_net "Net-(U2-Pad8)")
   )
+  (module Capacitor_SMD:C_1206_3216Metric_Pad1.42x1.75mm_HandSolder (layer B.Cu)
+    (at 125.222 106.7165 270)
+    (descr "Capacitor SMD 1206 (3216 Metric), square (rectangular) end terminal, IPC_7351 nominal with elongated pad for handsoldering. (Body size source: http://www.tortai-tech.com/upload/download/2011102023233369053.pdf), generated with kicad-footprint-generator")
+    (tags "capacitor handsolder")
+    (attr smd)
+    (fp_text reference C4 (at 0 1.82 270) (layer B.SilkS)
+      (effects (font (size 1 1) (thickness 0.15)) (justify mirror))
+    )
+    (fp_text value C (at 0 -1.82 270) (layer B.Fab)
+      (effects (font (size 1 1) (thickness 0.15)) (justify mirror))
+    )
+    (fp_line (start -1.6 -0.8) (end -1.6 0.8) (layer B.Fab) (width 0.1))
+    (fp_line (start -1.6 0.8) (end 1.6 0.8) (layer B.Fab) (width 0.1))
+    (fp_line (start 1.6 0.8) (end 1.6 -0.8) (layer B.Fab) (width 0.1))
+    (fp_line (start 1.6 -0.8) (end -1.6 -0.8) (layer B.Fab) (width 0.1))
+    (fp_line (start -0.602064 0.91) (end 0.602064 0.91) (layer B.SilkS) (width 0.12))
+    (fp_line (start -0.602064 -0.91) (end 0.602064 -0.91) (layer B.SilkS) (width 0.12))
+    (fp_line (start -2.45 -1.12) (end -2.45 1.12) (layer B.CrtYd) (width 0.05))
+    (fp_line (start -2.45 1.12) (end 2.45 1.12) (layer B.CrtYd) (width 0.05))
+    (fp_line (start 2.45 1.12) (end 2.45 -1.12) (layer B.CrtYd) (width 0.05))
+    (fp_line (start 2.45 -1.12) (end -2.45 -1.12) (layer B.CrtYd) (width 0.05))
+    (fp_text user %R (at 0 0 270) (layer B.Fab)
+      (effects (font (size 0.8 0.8) (thickness 0.12)) (justify mirror))
+    )
+    (pad 1 smd roundrect (at -1.4875 0 270) (size 1.425 1.75) (layers B.Cu B.Paste B.Mask) (roundrect_rratio 0.175439)
+      (net 65 VDD))
+    (pad 2 smd roundrect (at 1.4875 0 270) (size 1.425 1.75) (layers B.Cu B.Paste B.Mask) (roundrect_rratio 0.175439)
+      (net 67 GND))
+    (model ${KISYS3DMOD}/Capacitor_SMD.3dshapes/C_1206_3216Metric.wrl
+      (at (xyz 0 0 0))
+      (scale (xyz 1 1 1))
+      (rotate (xyz 0 0 0))
+    )
+  )
   (module omron-relay:g6j-2p-y (layer F.Cu)
     (at 168.91 85.725 90)
@@
       (net 65 VDD))
     (model ${KISYS3DMOD}/Capacitor_SMD.3dshapes/CP_Elec_10x7.9.wrl
-      (at (xyz 0 0 0))
-      (scale (xyz 1 1 1))
-      (rotate (xyz 0 0 0))
-    )
-  )
-  (module Capacitor_SMD:C_1206_3216Metric_Pad1.42x1.75mm_HandSolder (layer B.Cu)
-    (at 125.222 106.68 270)
-    (descr "Capacitor SMD 1206 (3216 Metric), square (rectangular) end terminal, IPC_7351 nominal with elongated pad for handsoldering. (Body size source: http://www.tortai-tech.com/upload/download/2011102023233369053.pdf), generated with kicad-footprint-generator")
-    (tags "capacitor handsolder")
-    (attr smd)
-    (fp_text reference C1 (at 0 1.82 270) (layer B.SilkS)
-      (effects (font (size 1 1) (thickness 0.15)) (justify mirror))
-    )
-    (fp_text value C (at 0 -1.82 270) (layer B.Fab)
-      (effects (font (size 1 1) (thickness 0.15)) (justify mirror))
-    )
-    (fp_text user %R (at 0 0 270) (layer B.Fab)
-      (effects (font (size 0.8 0.8) (thickness 0.12)) (justify mirror))
-    )
-    (fp_line (start 2.45 -1.12) (end -2.45 -1.12) (layer B.CrtYd) (width 0.05))
-    (fp_line (start 2.45 1.12) (end 2.45 -1.12) (layer B.CrtYd) (width 0.05))
-    (fp_line (start -2.45 1.12) (end 2.45 1.12) (layer B.CrtYd) (width 0.05))
-    (fp_line (start -2.45 -1.12) (end -2.45 1.12) (layer B.CrtYd) (width 0.05))
-    (fp_line (start -0.602064 -0.91) (end 0.602064 -0.91) (layer B.SilkS) (width 0.12))
-    (fp_line (start -0.602064 0.91) (end 0.602064 0.91) (layer B.SilkS) (width 0.12))
-    (fp_line (start 1.6 -0.8) (end -1.6 -0.8) (layer B.Fab) (width 0.1))
-    (fp_line (start 1.6 0.8) (end 1.6 -0.8) (layer B.Fab) (width 0.1))
-    (fp_line (start -1.6 0.8) (end 1.6 0.8) (layer B.Fab) (width 0.1))
-    (fp_line (start -1.6 -0.8) (end -1.6 0.8) (layer B.Fab) (width 0.1))
-    (pad 2 smd roundrect (at 1.4875 0 270) (size 1.425 1.75) (layers B.Cu B.Paste B.Mask) (roundrect_rratio 0.175439)
-      (net 67 GND))
-    (pad 1 smd roundrect (at -1.4875 0 270) (size 1.425 1.75) (layers B.Cu B.Paste B.Mask) (roundrect_rratio 0.175439)
-      (net 65 VDD))
-    (model ${KISYS3DMOD}/Capacitor_SMD.3dshapes/C_1206_3216Metric.wrl
       (at (xyz 0 0 0))
       (scale (xyz 1 1 1))
@@
       (effects (font (size 1 1) (thickness 0.15)))
     )
-    (pad 1 np_thru_hole circle (at 0 0) (size 3.2 3.2) (drill 3.2) (layers *.Cu *.Mask))
+    (pad 1 thru_hole circle (at 0 0) (size 6.1 6.1) (drill 3.05) (layers *.Cu *.Mask))
   )
   (module MountingHole:MountingHole_3.2mm_M3_DIN965 (layer F.Cu)
@@
       (effects (font (size 1 1) (thickness 0.15)))
     )
-    (pad 1 np_thru_hole circle (at 0 0) (size 3.2 3.2) (drill 3.2) (layers *.Cu *.Mask))
+    (pad 1 thru_hole circle (at 0 0) (size 6.1 6.1) (drill 3.05) (layers *.Cu *.Mask))
   )
   (module MountingHole:MountingHole_3.2mm_M3_DIN965 (layer F.Cu)
@@
       (effects (font (size 1 1) (thickness 0.15)))
     )
-    (pad 1 np_thru_hole circle (at 0 0) (size 3.2 3.2) (drill 3.2) (layers *.Cu *.Mask))
+    (pad "" thru_hole circle (at 0 0) (size 6.1 6.1) (drill 3.05) (layers *.Cu *.Mask))
   )
   (module MountingHole:MountingHole_3.2mm_M3_DIN965 (layer F.Cu)
@@
       (effects (font (size 1 1) (thickness 0.15)))
     )
-    (pad 1 np_thru_hole circle (at 0 0) (size 3.2 3.2) (drill 3.2) (layers *.Cu *.Mask))
+    (pad 1 thru_hole circle (at 0 0) (size 6.1 6.1) (drill 3.05) (layers *.Cu *.Mask))
   )
   (module MountingHole:MountingHole_3.2mm_M3_DIN965 (layer F.Cu)
@@
       (effects (font (size 1 1) (thickness 0.15)))
     )
-    (pad 1 np_thru_hole circle (at 0 0) (size 3.2 3.2) (drill 3.2) (layers *.Cu *.Mask))
+    (pad 1 thru_hole circle (at 0 0) (size 6.1 6.1) (drill 3.05) (layers *.Cu *.Mask))
   )
   (module Connector_Molex:Molex_KK-254_AE-6410-06A_1x06_P2.54mm_Vertical (layer F.Cu)
@@
     )
   )
+  (gr_text v3.0 (at 93.218 80.518) (layer F.SilkS)
+    (effects (font (size 1.5 1.5) (thickness 0.1778)) (justify left))
+  )
+  (gr_text v3.0 (at 98.298 80.518) (layer B.SilkS)
+    (effects (font (size 1.5 1.5) (thickness 0.1778)) (justify left mirror))
+  )
+  (gr_text "Input Selector v3.0" (at 170.434 78.232) (layer B.SilkS)
+    (effects (font (size 1.5 1.5) (thickness 0.1778)) (justify left mirror))
+  )
+  (gr_text "Input Selector v3.0" (at 147.828 121.158) (layer F.SilkS)
+    (effects (font (size 1.5 1.5) (thickness 0.1778)) (justify left))
+  )
   (gr_text - (at 100.584 102.108 90) (layer F.SilkS)
