File: PCBs/mdac-attenuator/mdac-attenuator.sch (KiCad schematic (older format))
At the start: 34 parts, among them J1 Conn_01x06_Male, J2 Conn_01x06_Male, U1 AD8620, U2 DAC8812ICPWG4

Commit message: adding BoMs, images and small design updates
Parts:
- C1A1, C1B1: footprint Resistor_SMD:R_0805_2012Metric_Pad1.15x1.40mm_HandSolder -> Capacitor_SMD:C_0805_2012Metric_Pad1.15x1.40mm_HandSolder
- C3, C4, C6: footprint Resistor_SMD:R_1206_3216Metric_Pad1.42x1.75mm_HandSolder -> Capacitor_SMD:C_1206_3216Metric_Pad1.42x1.75mm_HandSolder
Changed lines of the file:
@@
 F 0 "C4" H 4865 1746 50  0000 L CNN
 F 1 "C" H 4865 1655 50  0000 L CNN
-F 2 "Resistor_SMD:R_1206_3216Metric_Pad1.42x1.75mm_HandSolder" H 4788 1550 50  0001 C CNN
+F 2 "Capacitor_SMD:C_1206_3216Metric_Pad1.42x1.75mm_HandSolder" H 4788 1550 50  0001 C CNN
 F 3 "~" H 4750 1700 50  0001 C CNN
 	1    4750 1700
@@
 F 0 "C3" H 4865 1246 50  0000 L CNN
 F 1 "C" H 4865 1155 50  0000 L CNN
-F 2 "Resistor_SMD:R_1206_3216Metric_Pad1.42x1.75mm_HandSolder" H 4788 1050 50  0001 C CNN
+F 2 "Capacitor_SMD:C_1206_3216Metric_Pad1.42x1.75mm_HandSolder" H 4788 1050 50  0001 C CNN
 F 3 "~" H 4750 1200 50  0001 C CNN
 	1    4750 1200
@@
 F 0 "C1B1" H 7265 3196 50  0000 L CNN
 F 1 "2pF" H 7265 3105 50  0000 L CNN
-F 2 "Resistor_SMD:R_0805_2012Metric_Pad1.15x1.40mm_HandSolder" H 7188 3000 50  0001 C CNN
+F 2 "Capacitor_SMD:C_0805_2012Metric_Pad1.15x1.40mm_HandSolder" H 7188 3000 50  0001 C CNN
 F 3 "~" H 7150 3150 50  0001 C CNN
 	1    7150 3150
@@
 F 0 "C6" H 1465 1496 50  0000 L CNN
 F 1 "C" H 1465 1405 50  0000 L CNN
-F 2 "Resistor_SMD:R_1206_3216Metric_Pad1.42x1.75mm_HandSolder" H 1388 1300 50  0001 C CNN
+F 2 "Capacitor_SMD:C_1206_3216Metric_Pad1.42x1.75mm_HandSolder" H 1388 1300 50  0001 C CNN
 F 3 "~" H 1350 1450 50  0001 C CNN
 	1    1350 1450
@@
 F 0 "C1A1" H 7265 4796 50  0000 L CNN
 F 1 "2pF" H 7265 4705 50  0000 L CNN
-F 2 "Resistor_SMD:R_0805_2012Metric_Pad1.15x1.40mm_HandSolder" H 7188 4600 50  0001 C CNN
+F 2 "Capacitor_SMD:C_0805_2012Metric_Pad1.15x1.40mm_HandSolder" H 7188 4600 50  0001 C CNN
 F 3 "~" H 7150 4750 50  0001 C CNN
 	1    7150 4750
