File: PCBs/mdac-attenuator/mdac-attenuator.sch (KiCad schematic (older format))
At the start: 34 parts, among them J1 Conn_01x06_Male, J2 Conn_01x06_Male, U1 AD8620, U2 DAC8812ICPWG4

Commit message: Misc updates to 3 PCBs
Parts:
- C5_SMD1: footprint Capacitor_SMD:CP_Elec_10x10 -> Capacitor_SMD:CP_Elec_8x10
Changed lines of the file:
@@
 F 0 "C5_SMD1" H 1868 1496 50  0000 L CNN
 F 1 "CP" H 1868 1405 50  0000 L CNN
-F 2 "Capacitor_SMD:CP_Elec_10x10" H 1788 1300 50  0001 C CNN
+F 2 "Capacitor_SMD:CP_Elec_8x10" H 1788 1300 50  0001 C CNN
 F 3 "~" H 1750 1450 50  0001 C CNN
 	1    1750 1450

Commit message: adding BoMs, images and small design updates (#4)
Parts:
- C1A1, C1B1: footprint Resistor_SMD:R_0805_2012Metric_Pad1.15x1.40mm_HandSolder -> Capacitor_SMD:C_0805_2012Metric_Pad1.15x1.40mm_HandSolder
- C4: renamed from C3; value C -> 100nF; footprint Resistor_SMD:R_1206_3216Metric_Pad1.42x1.75mm_HandSolder -> Capacitor_SMD:C_1206_3216Metric_Pad1.42x1.75mm_HandSolder
- C6: renamed from C4; value C -> 100nF; footprint Resistor_SMD:R_1206_3216Metric_Pad1.42x1.75mm_HandSolder -> Capacitor_SMD:C_1206_3216Metric_Pad1.42x1.75mm_HandSolder
- C7: renamed from C6; value C -> 100nF; footprint Resistor_SMD:R_1206_3216Metric_Pad1.42x1.75mm_HandSolder -> Capacitor_SMD:C_1206_3216Metric_Pad1.42x1.75mm_HandSolder
- U1: value AD8620 -> AD8599
- renumbered C1_SMD1 to C3_SMD1, C1_TH1 to C3_TH1
Changed lines of the file:
@@
 P 7600 3500
 F 0 "U1" H 7600 3867 50  0000 C CNN
-F 1 "AD8620" H 7600 3776 50  0000 C CNN
+F 1 "AD8599" H 7600 3776 50  0000 C CNN
 F 2 "Package_SO:SOIC-8_3.9x4.9mm_P1.27mm" H 7600 3500 50  0001 C CNN
 F 3 "http://www.analog.com/media/en/technical-documentation/data-sheets/AD8610_8620.pdf" H 7600 3500 50  0001 C CNN
@@
 P 7600 4400
 F 0 "U1" H 7600 4767 50  0000 C CNN
-F 1 "AD8620" H 7600 4676 50  0000 C CNN
+F 1 "AD8599" H 7600 4676 50  0000 C CNN
 F 2 "Package_SO:SOIC-8_3.9x4.9mm_P1.27mm" H 7600 4400 50  0001 C CNN
 F 3 "http://www.analog.com/media/en/technical-documentation/data-sheets/AD8610_8620.pdf" H 7600 4400 50  0001 C CNN
@@
 P 5250 1450
 F 0 "U1" H 5208 1496 50  0000 L CNN
-F 1 "AD8620" H 5208 1405 50  0000 L CNN
+F 1 "AD8599" H 5208 1405 50  0000 L CNN
 F 2 "Package_SO:SOIC-8_3.9x4.9mm_P1.27mm" H 5250 1450 50  0001 C CNN
 F 3 "http://www.analog.com/media/en/technical-documentation/data-sheets/AD8610_8620.pdf" H 5250 1450 50  0001 C CNN
@@
 $EndComp
 $Comp
-L Device:C C4
+L Device:C C6
 U 1 1 5C279BB9
 P 4750 1700
-F 0 "C4" H 4865 1746 50  0000 L CNN
-F 1 "C" H 4865 1655 50  0000 L CNN
-F 2 "Resistor_SMD:R_1206_3216Metric_Pad1.42x1.75mm_HandSolder" H 4788 1550 50  0001 C CNN
+F 0 "C6" H 4865 1746 50  0000 L CNN
+F 1 "100nF" H 4865 1655 50  0000 L CNN
+F 2 "Capacitor_SMD:C_1206_3216Metric_Pad1.42x1.75mm_HandSolder" H 4788 1550 50  0001 C CNN
 F 3 "~" H 4750 1700 50  0001 C CNN
 	1    4750 1700
@@
 $EndComp
 $Comp
-L Device:C C3
+L Device:C C4
 U 1 1 5C279C71
 P 4750 1200
-F 0 "C3" H 4865 1246 50  0000 L CNN
-F 1 "C" H 4865 1155 50  0000 L CNN
-F 2 "Resistor_SMD:R_1206_3216Metric_Pad1.42x1.75mm_HandSolder" H 4788 1050 50  0001 C CNN
+F 0 "C4" H 4865 1246 50  0000 L CNN
+F 1 "100nF" H 4865 1155 50  0000 L CNN
+F 2 "Capacitor_SMD:C_1206_3216Metric_Pad1.42x1.75mm_HandSolder" H 4788 1050 50  0001 C CNN
 F 3 "~" H 4750 1200 50  0001 C CNN
 	1    4750 1200
@@
 F 0 "C1B1" H 7265 3196 50  0000 L CNN
 F 1 "2pF" H 7265 3105 50  0000 L CNN
-F 2 "Resistor_SMD:R_0805_2012Metric_Pad1.15x1.40mm_HandSolder" H 7188 3000 50  0001 C CNN
+F 2 "Capacitor_SMD:C_0805_2012Metric_Pad1.15x1.40mm_HandSolder" H 7188 3000 50  0001 C CNN
 F 3 "~" H 7150 3150 50  0001 C CNN
 	1    7150 3150
@@
 $EndComp
 $Comp
-L Device:C C6
+L Device:C C7
 U 1 1 5C279CE6
 P 1350 1450
-F 0 "C6" H 1465 1496 50  0000 L CNN
-F 1 "C" H 1465 1405 50  0000 L CNN
-F 2 "Resistor_SMD:R_1206_3216Metric_Pad1.42x1.75mm_HandSolder" H 1388 1300 50  0001 C CNN
+F 0 "C7" H 1465 1496 50  0000 L CNN
+F 1 "100nF" H 1465 1405 50  0000 L CNN
+F 2 "Capacitor_SMD:C_1206_3216Metric_Pad1.42x1.75mm_HandSolder" H 1388 1300 50  0001 C CNN
 F 3 "~" H 1350 1450 50  0001 C CNN
 	1    1350 1450
@@
 F 0 "C1A1" H 7265 4796 50  0000 L CNN
 F 1 "2pF" H 7265 4705 50  0000 L CNN
-F 2 "Resistor_SMD:R_0805_2012Metric_Pad1.15x1.40mm_HandSolder" H 7188 4600 50  0001 C CNN
+F 2 "Capacitor_SMD:C_0805_2012Metric_Pad1.15x1.40mm_HandSolder" H 7188 4600 50  0001 C CNN
 F 3 "~" H 7150 4750 50  0001 C CNN
 	1    7150 4750
@@
 $EndComp
 $Comp
-L Device:CP C1_SMD1
+L Device:CP C3_SMD1
 U 1 1 5C279F46
 P 3950 1200
-F 0 "C1_SMD1" H 4068 1246 50  0000 L CNN
+F 0 "C3_SMD1" H 4068 1246 50  0000 L CNN
 F 1 "CP" H 4068 1155 50  0000 L CNN
 F 2 "Capacitor_SMD:CP_Elec_8x10" H 3988 1050 50  0001 C CNN
@@
 $EndComp
 $Comp
-L Device:CP C1_TH1
+L Device:CP C3_TH1
 U 1 1 5C279FDB
 P 4350 1200
-F 0 "C1_TH1" H 4468 1246 50  0000 L CNN
+F 0 "C3_TH1" H 4468 1246 50  0000 L CNN
 F 1 "CP" H 4468 1155 50  0000 L CNN
 F 2 "Capacitor_THT:CP_Radial_D10.0mm_P5.00mm" H 4388 1050 50  0001 C CNN
