File: PCBs/mdac-attenuator/mdac-attenuator.kicad_pcb (KiCad board)
At the start: 2 copper layers, 45.7 x 52.1 mm, 34 parts, among them J1 Conn_01x06_Male, J2 Conn_01x06_Male, U1 AD8620, U2 DAC8812ICPWG4

Commit message: adding BoMs, images and small design updates (#4)
Parts:
- removed C3: C, Resistor_SMD:R_1206_3216Metric_Pad1.42x1.75mm_HandSolder
- added C7: 100nF, Capacitor_SMD:C_1206_3216Metric_Pad1.42x1.75mm_HandSolder, B.Cu at (146.1, 111.5)
- C1A1, C1B1: footprint Resistor_SMD:R_0805_2012Metric_Pad1.15x1.40mm_HandSolder -> Capacitor_SMD:C_0805_2012Metric_Pad1.15x1.40mm_HandSolder
- C4, C6: value C -> 100nF; footprint Resistor_SMD:R_1206_3216Metric_Pad1.42x1.75mm_HandSolder -> Capacitor_SMD:C_1206_3216Metric_Pad1.42x1.75mm_HandSolder
- U1: value AD8620 -> AD8599
- moved C6 11.8 mm to (144.8, 99.8)
- moved C4 4.63 mm to (147.3, 95.9)
- renumbered C1_SMD1 to C3_SMD1, C1_TH1 to C3_TH1
Connections:
- C4 pad 1: GNDA -> +15V
- C4 pad 2: -15V -> GNDA
- C6 pad 1: VDD -> GNDA
- C6 pad 2: GNDA -> -15V
Other:
- board text added: "C3"
