File: PCBs/rca-panel/rca-panel.kicad_pcb (KiCad board)
At the start: 2 copper layers, 141 x 52.1 mm, 25 parts

Commit message: updating 3 PCBs to kicad
Parts:
- added LOGO1: Logo_Open_Hardware_Small, Symbol:OSHW-Logo2_7.3x6mm_SilkScreen, F.Cu at (73.0, 67.9)
- added LOGO2: Logo_Open_Hardware_Small, Symbol:OSHW-Logo2_7.3x6mm_SilkScreen, B.Cu at (73.0, 67.9)
- moved MH5 0.63 mm to (189.9, 67.9)
- moved MH6 0.63 mm to (189.9, 111.1)
- moved MH7 0.63 mm to (108.6, 111.1)
- moved MH8 0.63 mm to (108.6, 67.9)
Other:
- rule pad_to_mask_clearance: 0.2 -> 0.0508
- board text added: "Designed by Max Williams"
- board text added: "IN1"
- board text added: "IN2"
- board text added: "IN3"
- board text added: "IN4"
- board text added: "IN5"
- board text added: "IN6"
- board text added: "OUT"
- board text added: "futuresharks@gmail.com"
- board text added: "github.com/FutureSharks/preamp-two"

Commit message: Add new text
Other:
- board text added: "RCA Panel v2.0"
Changed lines of the file:
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@@
   (general
     (thickness 1.6)
-    (drawings 28)
+    (drawings 30)
     (tracks 121)
     (zones 0)
@@
       (net 16 "Net-(IN6-Pad3)"))
   )
+  (gr_text "RCA Panel v2.0" (at 104.14 66.675) (layer B.SilkS)
+    (effects (font (size 1.5 1.5) (thickness 0.127)) (justify left mirror))
+  )
+  (gr_text "RCA Panel v2.0" (at 86.36 66.675) (layer F.SilkS)
+    (effects (font (size 1.5 1.5) (thickness 0.127)) (justify left))
+  )
   (gr_text "Designed by Max Williams" (at 101.6 111.125) (layer B.SilkS)
-    (effects (font (size 1.5 1.5) (thickness 0.2032)) (justify left mirror))
+    (effects (font (size 1.5 1.5) (thickness 0.127)) (justify left mirror))
   )
   (gr_text github.com/FutureSharks/preamp-two (at 184.785 111.125) (layer B.SilkS)
-    (effects (font (size 1.5 1.5) (thickness 0.2032)) (justify left mirror))
+    (effects (font (size 1.5 1.5) (thickness 0.127)) (justify left mirror))
   )
   (gr_text futuresharks@gmail.com (at 186.69 76.2 90) (layer B.SilkS)
-    (effects (font (size 1.5 1.5) (thickness 0.2032)) (justify left mirror))
+    (effects (font (size 1.5 1.5) (thickness 0.127)) (justify left mirror))
   )
   (gr_text "Designed by Max Williams" (at 71.755 111.125) (layer F.SilkS)
-    (effects (font (size 1.5 1.5) (thickness 0.2032)) (justify left))
+    (effects (font (size 1.5 1.5) (thickness 0.127)) (justify left))
   )
   (gr_text github.com/FutureSharks/preamp-two (at 113.665 111.125) (layer F.SilkS)
-    (effects (font (size 1.5 1.5) (thickness 0.2032)) (justify left))
+    (effects (font (size 1.5 1.5) (thickness 0.127)) (justify left))
   )
   (gr_text futuresharks@gmail.com (at 186.69 103.505 90) (layer F.SilkS)
-    (effects (font (size 1.5 1.5) (thickness 0.2032)) (justify left))
+    (effects (font (size 1.5 1.5) (thickness 0.127)) (justify left))
   )
   (gr_text OUT (at 201.676 89.662) (layer B.SilkS)

Commit message: New RCA board (#7)
* updating PCB after creating new library for newer 805 RCAs

* fix for mounting holes
Parts:
- OUT_L1, OUT_R1, RCA_1_L1, RCA_1_R1, RCA_2_L1, RCA_2_R1, RCA_3_L1, RCA_3_R1, RCA_4_L1, RCA_4_R1, RCA_5_L1, RCA_5_R1, RCA_6_L1, RCA_6_R1: footprint rca-panel:cmc-805 -> rca-panel:cmc-805-new
Other:
- board text added: "RCA Panel v2.1"
- board text removed: "RCA Panel v2.0"
