File: PCBs/rca-panel/rca-panel.sch (KiCad schematic (older format))
At the start: 25 parts

Commit message: updating 3 PCBs to kicad
Parts:
- added LOGO1, LOGO2: Logo_Open_Hardware_Small, Symbol:OSHW-Logo2_7.3x6mm_SilkScreen, symbol Graphic:Logo_Open_Hardware_Small
Changed lines of the file:
@@
 	8150 3600 8150 3100
 Connection ~ 8150 3100
+$Comp
+L Graphic:Logo_Open_Hardware_Small LOGO1
+U 1 1 5C327FDF
+P 2950 4700
+F 0 "LOGO1" H 2950 4975 50  0001 C CNN
+F 1 "Logo_Open_Hardware_Small" H 2950 4475 50  0001 C CNN
+F 2 "Symbol:OSHW-Logo2_7.3x6mm_SilkScreen" H 2950 4700 50  0001 C CNN
+F 3 "~" H 2950 4700 50  0001 C CNN
+	1    2950 4700
+	1    0    0    -1
+$EndComp
+$Comp
+L Graphic:Logo_Open_Hardware_Small LOGO2
+U 1 1 5C2A8D32
+P 3450 4700
+F 0 "LOGO2" H 3450 4975 50  0001 C CNN
+F 1 "Logo_Open_Hardware_Small" H 3450 4475 50  0001 C CNN
+F 2 "Symbol:OSHW-Logo2_7.3x6mm_SilkScreen" H 3450 4700 50  0001 C CNN
+F 3 "~" H 3450 4700 50  0001 C CNN
+	1    3450 4700
+	1    0    0    -1
+$EndComp
 $EndSCHEMATC

Commit message: New RCA board (#7)
* updating PCB after creating new library for newer 805 RCAs

* fix for mounting holes
Parts:
- OUT_L1, OUT_R1, RCA_1_L1, RCA_1_R1, RCA_2_L1, RCA_2_R1, RCA_3_L1, RCA_3_R1, RCA_4_L1, RCA_4_R1, RCA_5_L1, RCA_5_R1, RCA_6_L1, RCA_6_R1: footprint rca-panel:cmc-805 -> rca-panel:cmc-805-new
Changed lines of the file:
@@
 F 0 "RCA_1_L1" H 2849 2476 50  0000 L CNN
 F 1 "Conn_Coaxial" H 2849 2385 50  0000 L CNN
-F 2 "rca-panel:cmc-805" H 2750 2500 50  0001 C CNN
+F 2 "rca-panel:cmc-805-new" H 2750 2500 50  0001 C CNN
 F 3 " ~" H 2750 2500 50  0001 C CNN
 	1    2750 2500
@@
 F 0 "RCA_1_R1" H 2849 2876 50  0000 L CNN
 F 1 "Conn_Coaxial" H 2849 2785 50  0000 L CNN
-F 2 "rca-panel:cmc-805" H 2750 2900 50  0001 C CNN
+F 2 "rca-panel:cmc-805-new" H 2750 2900 50  0001 C CNN
 F 3 " ~" H 2750 2900 50  0001 C CNN
 	1    2750 2900
@@
 F 0 "RCA_2_L1" H 3649 2476 50  0000 L CNN
 F 1 "Conn_Coaxial" H 3649 2385 50  0000 L CNN
-F 2 "rca-panel:cmc-805" H 3550 2500 50  0001 C CNN
+F 2 "rca-panel:cmc-805-new" H 3550 2500 50  0001 C CNN
 F 3 " ~" H 3550 2500 50  0001 C CNN
 	1    3550 2500
@@
 F 0 "RCA_2_R1" H 3649 2876 50  0000 L CNN
 F 1 "Conn_Coaxial" H 3649 2785 50  0000 L CNN
-F 2 "rca-panel:cmc-805" H 3550 2900 50  0001 C CNN
+F 2 "rca-panel:cmc-805-new" H 3550 2900 50  0001 C CNN
 F 3 " ~" H 3550 2900 50  0001 C CNN
 	1    3550 2900
@@
 F 0 "RCA_3_L1" H 4449 2476 50  0000 L CNN
 F 1 "Conn_Coaxial" H 4449 2385 50  0000 L CNN
-F 2 "rca-panel:cmc-805" H 4350 2500 50  0001 C CNN
+F 2 "rca-panel:cmc-805-new" H 4350 2500 50  0001 C CNN
 F 3 " ~" H 4350 2500 50  0001 C CNN
 	1    4350 2500
@@
 F 0 "RCA_3_R1" H 4449 2876 50  0000 L CNN
 F 1 "Conn_Coaxial" H 4449 2785 50  0000 L CNN
-F 2 "rca-panel:cmc-805" H 4350 2900 50  0001 C CNN
+F 2 "rca-panel:cmc-805-new" H 4350 2900 50  0001 C CNN
 F 3 " ~" H 4350 2900 50  0001 C CNN
 	1    4350 2900
@@
 F 0 "RCA_4_L1" H 5249 2476 50  0000 L CNN
 F 1 "Conn_Coaxial" H 5249 2385 50  0000 L CNN
-F 2 "rca-panel:cmc-805" H 5150 2500 50  0001 C CNN
+F 2 "rca-panel:cmc-805-new" H 5150 2500 50  0001 C CNN
 F 3 " ~" H 5150 2500 50  0001 C CNN
 	1    5150 2500
@@
 F 0 "RCA_4_R1" H 5249 2876 50  0000 L CNN
 F 1 "Conn_Coaxial" H 5249 2785 50  0000 L CNN
-F 2 "rca-panel:cmc-805" H 5150 2900 50  0001 C CNN
+F 2 "rca-panel:cmc-805-new" H 5150 2900 50  0001 C CNN
 F 3 " ~" H 5150 2900 50  0001 C CNN
 	1    5150 2900
@@
 F 0 "RCA_5_L1" H 6049 2476 50  0000 L CNN
 F 1 "Conn_Coaxial" H 6049 2385 50  0000 L CNN
-F 2 "rca-panel:cmc-805" H 5950 2500 50  0001 C CNN
+F 2 "rca-panel:cmc-805-new" H 5950 2500 50  0001 C CNN
 F 3 " ~" H 5950 2500 50  0001 C CNN
 	1    5950 2500
@@
 F 0 "RCA_5_R1" H 6049 2876 50  0000 L CNN
 F 1 "Conn_Coaxial" H 6049 2785 50  0000 L CNN
-F 2 "rca-panel:cmc-805" H 5950 2900 50  0001 C CNN
+F 2 "rca-panel:cmc-805-new" H 5950 2900 50  0001 C CNN
 F 3 " ~" H 5950 2900 50  0001 C CNN
 	1    5950 2900
@@
 F 0 "RCA_6_L1" H 6849 2476 50  0000 L CNN
 F 1 "Conn_Coaxial" H 6849 2385 50  0000 L CNN
-F 2 "rca-panel:cmc-805" H 6750 2500 50  0001 C CNN
+F 2 "rca-panel:cmc-805-new" H 6750 2500 50  0001 C CNN
 F 3 " ~" H 6750 2500 50  0001 C CNN
 	1    6750 2500
@@
 F 0 "RCA_6_R1" H 6849 2876 50  0000 L CNN
 F 1 "Conn_Coaxial" H 6849 2785 50  0000 L CNN
-F 2 "rca-panel:cmc-805" H 6750 2900 50  0001 C CNN
+F 2 "rca-panel:cmc-805-new" H 6750 2900 50  0001 C CNN
 F 3 " ~" H 6750 2900 50  0001 C CNN
 	1    6750 2900
@@
 F 0 "OUT_L1" H 8249 2476 50  0000 L CNN
 F 1 "Conn_Coaxial" H 8249 2385 50  0000 L CNN
-F 2 "rca-panel:cmc-805" H 8150 2500 50  0001 C CNN
+F 2 "rca-panel:cmc-805-new" H 8150 2500 50  0001 C CNN
 F 3 " ~" H 8150 2500 50  0001 C CNN
 	1    8150 2500
@@
 F 0 "OUT_R1" H 8249 2876 50  0000 L CNN
 F 1 "Conn_Coaxial" H 8249 2785 50  0000 L CNN
-F 2 "rca-panel:cmc-805" H 8150 2900 50  0001 C CNN
+F 2 "rca-panel:cmc-805-new" H 8150 2900 50  0001 C CNN
 F 3 " ~" H 8150 2900 50  0001 C CNN
 	1    8150 2900
